Commit message: add controller and collision box

File: emu_description/urdf/emu.xacro (robot description, xacro)
@@ -1,5 +1,12 @@
 <?xml version="1.0"?>
-<robot name="emu_manipulator" xmlns:xacro="http://www.ros.org/wiki/xacro">
+<robot name="emu" xmlns:xacro="http://www.ros.org/wiki/xacro">
+     <gazebo>
+        <plugin name="gazebo_ros_control" filename="libgazebo_ros_control.so">
+            <robotNamespace>/emu</robotNamespace>
+        </plugin>
+    </gazebo>
     <xacro:include filename="$(find emu_description)/urdf/emu.gazebo"/>
+    <xacro:include filename="$(find emu_description)/urdf/camera.xacro"/>
+    <xacro:emu_cam parent = "link_4" offset_from_parent = "-0.039 0.109 0.444 " rotate_from_parent = "1.57075 0 3.14159265359"/>
 <!--=================== LINKS ========================-->
     <link name="world"/>
@@ -169,4 +176,5 @@
         <axis xyz = "0 0 1"/>
         <limit lower = "-3.1066" upper = "3.1066" effort = "50" velocity = "10"/>
+        <dynamics damping="0.7"/>
     </joint>
     <joint name="joint_2" type="revolute">
@@ -176,4 +184,5 @@
         <limit lower = "-2.917" upper = "1.703" effort = "50" velocity = "10"/>
         <origin rpy="1.57075 0 0" xyz = "0.12596 0 0.30767"/>
+        <dynamics damping="0.8"/>
     </joint>
     <joint name="joint_3" type="revolute">
@@ -183,4 +192,5 @@
         <limit lower = "-1.4312" upper = "4.1190" effort = "50" velocity = "10"/>
         <origin rpy="0 0 1.57075" xyz = "0 0.4 0"/>
+        <dynamics damping="0.7"/>
     </joint>
     <joint name="joint_4" type="revolute">
@@ -190,4 +200,5 @@
         <limit lower = "-3.1067" upper = "3.1067" effort = "50" velocity = "10"/>
         <origin rpy="1.57075 0 0" xyz = "0.05 0 0"/>
+        <dynamics damping="0.7"/>
     </joint>
     <joint name="joint_5" type="revolute">
@@ -197,4 +208,5 @@
         <limit lower = "-3.1067" upper = "3.1067" effort = "50" velocity = "10"/>
         <origin rpy="-1.57075 0 0" xyz = "0 0 0.466"/>
+        <dynamics damping="0.2"/>
     </joint>
     <joint name="joint_6" type="revolute">
@@ -204,4 +216,65 @@
         <limit lower = "-3.1067" upper = "3.1067" effort = "50" velocity = "10"/>
         <origin rpy="1.57075 0 0" xyz = "0 0 0"/>
-    </joint>
+        <dynamics damping="0.2"/>
+    </joint>
+    <transmission name="tran1">
+        <type>transmission_interface/SimpleTransmission</type>
+        <joint name="joint_1">
+            <hardwareInterface>hardware_interface/EffortJointInterface</hardwareInterface>
+        </joint>
+        <actuator name="motor1">
+            <hardwareInterface>hardware_interface/EffortJointInterface</hardwareInterface>
+            <mechanicalReduction>1</mechanicalReduction>
+        </actuator>
+    </transmission>
+    <transmission name="tran2">
+        <type>transmission_interface/SimpleTransmission</type>
+        <joint name="joint_2">
+            <hardwareInterface>hardware_interface/EffortJointInterface</hardwareInterface>
+        </joint>
+        <actuator name="motor2">
+            <hardwareInterface>hardware_interface/EffortJointInterface</hardwareInterface>
+            <mechanicalReduction>1</mechanicalReduction>
+        </actuator>
+    </transmission>
+    <transmission name="tran3">
+        <type>transmission_interface/SimpleTransmission</type>
+        <joint name="joint_3">
+            <hardwareInterface>hardware_interface/EffortJointInterface</hardwareInterface>
+        </joint>
+        <actuator name="motor3">
+            <hardwareInterface>hardware_interface/EffortJointInterface</hardwareInterface>
+            <mechanicalReduction>1</mechanicalReduction>
+        </actuator>
+    </transmission>
+    <transmission name="tran4">
+        <type>transmission_interface/SimpleTransmission</type>
+        <joint name="joint_4">
+            <hardwareInterface>hardware_interface/EffortJointInterface</hardwareInterface>
+        </joint>
+        <actuator name="motor4">
+            <hardwareInterface>hardware_interface/EffortJointInterface</hardwareInterface>
+            <mechanicalReduction>1</mechanicalReduction>
+        </actuator>
+    </transmission>
+    <transmission name="tran5">
+        <type>transmission_interface/SimpleTransmission</type>
+        <joint name="joint_5">
+            <hardwareInterface>hardware_interface/EffortJointInterface</hardwareInterface>
+        </joint>
+        <actuator name="motor5">
+            <hardwareInterface>hardware_interface/EffortJointInterface</hardwareInterface>
+            <mechanicalReduction>1</mechanicalReduction>
+        </actuator>
+    </transmission>
+    <transmission name="tran6">
+        <type>transmission_interface/SimpleTransmission</type>
+        <joint name="joint_6">
+            <hardwareInterface>hardware_interface/EffortJointInterface</hardwareInterface>
+        </joint>
+        <actuator name="motor6">
+            <hardwareInterface>hardware_interface/EffortJointInterface</hardwareInterface>
+            <mechanicalReduction>1</mechanicalReduction>
+        </actuator>
+    </transmission>
 </robot>

Commit message: add workspace visual

File: emu_description/urdf/emu.xacro (robot description, xacro)
@@ -20,13 +20,17 @@
 			<origin xyz="0 0 0"/>
 			<geometry>
-				<mesh filename="$(find emu_description)/meshes/work_space.STL" scale="1 1 1"/>
-			</geometry>
-		</collision>
-        <visual>
-            <geometry>
-                <mesh filename="$(find emu_description)/meshes/work_space.STL" scale="1 1 1"/>
-            </geometry>
-        </visual>
-    </link>
+				<mesh filename="$(find emu_description)/meshes/work_plane.STL" scale="1 1 1"/>
+			</geometry>
+		</collision>
+        <visual>
+            <origin xyz = "0 0 0" rpy = "0 0 0"/>
+            <geometry>
+                <mesh filename="$(find emu_description)/meshes/work_plane.STL" scale="1 1 1"/>
+            </geometry>
+        </visual>
+    </link>
+    <gazebo reference="workspace">
+        <!-- <material>workspace</material> -->
+    </gazebo>
     <link name="base_link">
 		<inertial>

Commit message: add embedded talker node (not yet finished)

File: emu_description/urdf/emu.xacro (robot description, xacro)
@@ -20,5 +20,5 @@
 			<origin xyz="0 0 0"/>
 			<geometry>
-				<mesh filename="$(find emu_description)/meshes/work_plane.STL" scale="1 1 1"/>
+				<mesh filename="package://emu_description/meshes/work_plane.STL" scale="1 1 1"/>
 			</geometry>
 		</collision>
@@ -26,6 +26,9 @@
             <origin xyz = "0 0 0" rpy = "0 0 0"/>
             <geometry>
-                <mesh filename="$(find emu_description)/meshes/work_plane.STL" scale="1 1 1"/>
-            </geometry>
+                <mesh filename="package://emu_description/meshes/work_plane.STL" scale="1 1 1"/>
+            </geometry>
+            <material name="Grey">
+                <color rgba="0.7 0.7 0.7 1"/>
+            </material>
         </visual>
     </link>
@@ -42,12 +45,14 @@
 			<origin xyz="0 0 0"/>
 			<geometry>
-				<mesh filename="$(find emu_description)/meshes/collision/Base_link_c.STL" scale="1 1 1"/>
-			</geometry>
-		</collision>
-        <visual>
-            <geometry>
-                <mesh filename="$(find emu_description)/meshes/Base_link.STL" scale="1 1 1"/>
-            </geometry>
-        </visual>
+				<mesh filename="package://emu_description/meshes/collision/Base_link_c.STL" scale="1 1 1"/>
+			</geometry>
+		</collision>
+        <visual>
+            <geometry>
+                <mesh filename="package://emu_description/meshes/Base_link.STL" scale="1 1 1"/>
+            </geometry>
+            <material name="Grey">
+        <color rgba="0.7 0.7 0.7 1"/>
+    </material></visual>
     </link>
     <link name="link_1">
@@ -60,13 +65,15 @@
 			<origin xyz="0 0 0"/>
 			<geometry>
-				<mesh filename="$(find emu_description)/meshes/collision/Link1_c.STL" scale="1 1 1"/>
-			</geometry>
-		</collision>
-        <visual>
-            <geometry>
-                <mesh filename="$(find emu_description)/meshes/Link1.STL" scale="1 1 1"/>
+				<mesh filename="package://emu_description/meshes/collision/Link1_c.STL" scale="1 1 1"/>
+			</geometry>
+		</collision>
+        <visual>
+            <geometry>
+                <mesh filename="package://emu_description/meshes/Link1.STL" scale="1 1 1"/>
             </geometry>
             <origin rpy="1.57075 0 0" xyz = "0.12596 0 0.30767"/>
-        </visual>
+            <material name="Grey">
+        <color rgba="0.7 0.7 0.7 1"/>
+    </material></visual>
     </link>
     <link name="link_2">
@@ -79,13 +86,15 @@
 			<origin xyz="0 0 0"/>
 			<geometry>
-				<mesh filename="$(find emu_description)/meshes/collision/Link2_c.STL" scale="1 1 1"/>
-			</geometry>
-		</collision>
-        <visual>
-            <geometry>
-                <mesh filename="$(find emu_description)/meshes/Link2.STL" scale="1 1 1"/>
+				<mesh filename="package://emu_description/meshes/collision/Link2_c.STL" scale="1 1 1"/>
+			</geometry>
+		</collision>
+        <visual>
+            <geometry>
+                <mesh filename="package://emu_description/meshes/Link2.STL" scale="1 1 1"/>
             </geometry>
             <origin rpy="0 0 1.57075" xyz = "0 0.4 0"/>
-        </visual>
+            <material name="Grey">
+        <color rgba="0.7 0.7 0.7 1"/>
+    </material></visual>
     </link>
     <link name="link_3">
@@ -98,13 +107,15 @@
 			<origin xyz="0 0 0"/>
 			<geometry>
-				<mesh filename="$(find emu_description)/meshes/collision/Link3_c.STL" scale="1 1 1"/>
-			</geometry>
-		</collision>
-        <visual>
-            <geometry>
-                <mesh filename="$(find emu_description)/meshes/Link3.STL" scale="1 1 1"/>
+				<mesh filename="package://emu_description/meshes/collision/Link3_c.STL" scale="1 1 1"/>
+			</geometry>
+		</collision>
+        <visual>
+            <geometry>
+                <mesh filename="package://emu_description/meshes/Link3.STL" scale="1 1 1"/>
             </geometry>
             <origin rpy="1.57075 0 0" xyz = "0.05 0 0"/>
-        </visual>
+            <material name="Grey">
+        <color rgba="0.7 0.7 0.7 1"/>
+    </material></visual>
     </link>
     <link name="link_4">
@@ -117,13 +128,15 @@
 			<origin xyz="0 0 0"/>
 			<geometry>
-				<mesh filename="$(find emu_description)/meshes/collision/Link4_c.STL" scale="1 1 1"/>
-			</geometry>
-		</collision>
-        <visual>
-            <geometry>
-                <mesh filename="$(find emu_description)/meshes/Link4.STL" scale="1 1 1"/>
+				<mesh filename="package://emu_description/meshes/collision/Link4_c.STL" scale="1 1 1"/>
+			</geometry>
+		</collision>
+        <visual>
+            <geometry>
+                <mesh filename="package://emu_description/meshes/Link4.STL" scale="1 1 1"/>
             </geometry>
             <origin rpy="-1.57075 0 0" xyz = "0 0 0.466"/>
-        </visual>
+            <material name="Grey">
+        <color rgba="0.7 0.7 0.7 1"/>
+    </material></visual>
     </link>
     <link name="link_5">
@@ -136,13 +149,15 @@
 			<origin xyz="0 0 0"/>
 			<geometry>
-				<mesh filename="$(find emu_description)/meshes/collision/Link5_c.STL" scale="1 1 1"/>
-			</geometry>
-		</collision>
-        <visual>
-            <geometry>
-                <mesh filename="$(find emu_description)/meshes/Link5.STL" scale="1 1 1"/>
+				<mesh filename="package://emu_description/meshes/collision/Link5_c.STL" scale="1 1 1"/>
+			</geometry>
+		</collision>
+        <visual>
+            <geometry>
+                <mesh filename="package://emu_description/meshes/Link5.STL" scale="1 1 1"/>
             </geometry>
             <origin rpy="1.57075 0 0" xyz = "0 0 0"/>
-        </visual>
+            <material name="Grey">
+        <color rgba="0.7 0.7 0.7 1"/>
+    </material></visual>
     </link>
     <link name="link_6">
@@ -155,5 +170,5 @@
 			<origin xyz="0 0 0"/>
 			<geometry>
-				<mesh filename="$(find emu_description)/meshes/collision/Link6_c.STL" scale="1 1 1"/>
+				<mesh filename="package://emu_description/meshes/collision/Link6_c.STL" scale="1 1 1"/>
 			</geometry>
 		</collision>
@@ -163,5 +178,7 @@
             </geometry>
             <origin rpy="0 0 0" xyz = "0 0 0.121"/>
-        </visual>
+            <material name="Grey">
+        <color rgba="0.7 0.7 0.7 1"/>
+    </material></visual>
     </link>
 <!--=================== JOINTS ========================-->
@@ -180,5 +197,5 @@
         <axis xyz = "0 0 1"/>
         <limit lower = "-3.1066" upper = "3.1066" effort = "1000" velocity = "1000"/>
-        <dynamics damping="0.7"/>
+        <dynamics damping="0.1"/>
     </joint>
     <joint name="joint_2" type="revolute">
@@ -188,5 +205,5 @@
         <limit lower = "-2.917" upper = "1.703" effort = "1000" velocity = "1000"/>
         <origin rpy="1.57075 0 0" xyz = "0.12596 0 0.30767"/>
-        <dynamics damping="1"/>
+        <dynamics damping="0.1"/>
     </joint>
     <joint name="joint_3" type="revolute">
@@ -196,5 +213,5 @@
         <limit lower = "-1.4312" upper = "4.1190" effort = "1000" velocity = "1000"/>
         <origin rpy="0 0 1.57075" xyz = "0 0.4 0"/>
-        <dynamics damping="1"/>
+        <dynamics damping="0.1"/>
     </joint>
     <joint name="joint_4" type="revolute">
@@ -204,5 +221,5 @@
         <limit lower = "-3.1067" upper = "3.1067" effort = "1000" velocity = "1000"/>
         <origin rpy="1.57075 0 0" xyz = "0.05 0 0"/>
-        <dynamics damping="0.7"/>
+        <dynamics damping="0.03"/>
     </joint>
     <joint name="joint_5" type="revolute">
@@ -212,5 +229,5 @@
         <limit lower = "-3.1067" upper = "3.1067" effort = "1000" velocity = "1000"/>
         <origin rpy="-1.57075 0 0" xyz = "0 0 0.466"/>
-        <dynamics damping="0.2"/>
+        <dynamics damping="0.01"/>
     </joint>
     <joint name="joint_6" type="revolute">

Commit message: add emu planner

File: emu_description/urdf/emu.xacro (robot description, xacro)
@@ -10,30 +10,5 @@
     <xacro:emu_cam parent = "link_4" offset_from_parent = "0.0 0.109 0.444 " rotate_from_parent = "0 0 1.57075"/>
 <!--=================== LINKS ========================-->
-    <link name="world"/>
-    <link name="workspace">
-        <inertial>
-			<origin xyz = "0 0 0"/>
-			<mass value = "10"/>
-			<inertia ixx = "0.02107003" iyy = "0.04864817" izz = "0.05239187" ixy = "0.00000013" ixz = "0.0149951" iyz = "-0.00000032"/>
-		</inertial>
-        <collision>
-			<origin xyz="0 0 0"/>
-			<geometry>
-				<mesh filename="package://emu_description/meshes/work_plane.STL" scale="1 1 1"/>
-			</geometry>
-		</collision>
-        <visual>
-            <origin xyz = "0 0 0" rpy = "0 0 0"/>
-            <geometry>
-                <mesh filename="package://emu_description/meshes/work_plane.STL" scale="1 1 1"/>
-            </geometry>
-            <material name="Grey">
-                <color rgba="0.7 0.7 0.7 1"/>
-            </material>
-        </visual>
-    </link>
-    <gazebo reference="workspace">
-        <!-- <material>workspace</material> -->
-    </gazebo>
+    <!-- <link name="world"/> -->
     <link name="base_link">
 		<inertial>
@@ -175,5 +150,5 @@
         <visual>
             <geometry>
-                <mesh filename="$(find emu_description)/meshes/Link6.STL" scale="1 1 1"/>
+                <mesh filename="package://emu_description/meshes/Link6.STL" scale="1 1 1"/>
             </geometry>
             <origin rpy="0 0 0" xyz = "0 0 0.121"/>
@@ -183,13 +158,9 @@
     </link>
 <!--=================== JOINTS ========================-->
-    <joint name="world_to_base" type="fixed">
+    <!-- <joint name="world_to_base" type="fixed">
         <parent link="world"/>
         <child link="base_link"/>
         <origin xyz = "0 0 0.001"/>
-    </joint>
-    <joint name="world_to_workspace" type="fixed">
-        <parent link="world"/>
-        <child link="workspace"/>
-    </joint>
+    </joint> -->
     <joint name="joint_1" type="revolute">
         <parent link="base_link"/>

Commit message: update urdf model

File: emu_description/urdf/emu.xacro (robot description, xacro)
@@ -28,6 +28,7 @@
             </geometry>
             <material name="Grey">
-        <color rgba="0.7 0.7 0.7 1"/>
-    </material></visual>
+                <color rgba="0.7 0.7 0.7 1"/>
+            </material>
+        </visual>
     </link>
     <link name="link_1">
@@ -49,6 +50,7 @@
             <origin rpy="1.57075 0 0" xyz = "0.12596 0 0.30767"/>
             <material name="Grey">
-        <color rgba="0.7 0.7 0.7 1"/>
-    </material></visual>
+                <color rgba="0.7 0.7 0.7 1"/>
+            </material>
+        </visual>
     </link>
     <link name="link_2">
@@ -70,6 +72,7 @@
             <origin rpy="0 0 1.57075" xyz = "0 0.4 0"/>
             <material name="Grey">
-        <color rgba="0.7 0.7 0.7 1"/>
-    </material></visual>
+                <color rgba="0.7 0.7 0.7 1"/>
+            </material>
+        </visual>
     </link>
     <link name="link_3">
@@ -91,6 +94,7 @@
             <origin rpy="1.57075 0 0" xyz = "0.05 0 0"/>
             <material name="Grey">
-        <color rgba="0.7 0.7 0.7 1"/>
-    </material></visual>
+                <color rgba="0.7 0.7 0.7 1"/>
+            </material>
+        </visual>
     </link>
     <link name="link_4">
@@ -112,6 +116,7 @@
             <origin rpy="-1.57075 0 0" xyz = "0 0 0.466"/>
             <material name="Grey">
-        <color rgba="0.7 0.7 0.7 1"/>
-    </material></visual>
+                <color rgba="0.7 0.7 0.7 1"/>
+            </material>
+        </visual>
     </link>
     <link name="link_5">
@@ -133,6 +138,7 @@
             <origin rpy="1.57075 0 0" xyz = "0 0 0"/>
             <material name="Grey">
-        <color rgba="0.7 0.7 0.7 1"/>
-    </material></visual>
+                <color rgba="0.7 0.7 0.7 1"/>
+            </material>
+        </visual>
     </link>
     <link name="link_6">
@@ -145,5 +151,5 @@
 			<origin xyz="0 0 0"/>
 			<geometry>
-				<mesh filename="package://emu_description/meshes/collision/Link6_c.STL" scale="1 1 1"/>
+				<mesh filename="package://emu_description/meshes/Link6.STL" scale="1 1 1"/>
 			</geometry>
 		</collision>
@@ -152,8 +158,29 @@
                 <mesh filename="package://emu_description/meshes/Link6.STL" scale="1 1 1"/>
             </geometry>
-            <origin rpy="0 0 0" xyz = "0 0 0.121"/>
-            <material name="Grey">
-        <color rgba="0.7 0.7 0.7 1"/>
-    </material></visual>
+            <material name="Grey">
+                <color rgba="0.7 0.7 0.7 1"/>
+            </material>
+        </visual>
+    </link>
+    <link name="tool">
+		<inertial>
+			<origin xyz = "-0.00016738 0 0.04413320"/>
+			<mass value = "0.43864195"/>
+			<inertia ixx = "0.00049965" iyy = "0.00043225" izz = "0.00020871" ixy = "0" ixz = "-0.00000204" iyz = "0"/>
+		</inertial>
+        <collision>
+			<origin xyz="0 0 0"/>
+			<geometry>
+				<mesh filename="package://emu_description/meshes/tool_joulin.STL" scale="1 1 1"/>
+			</geometry>
+		</collision>
+        <visual>
+            <geometry>
+                <mesh filename="package://emu_description/meshes/tool_joulin.STL" scale="1 1 1"/>
+            </geometry>
+            <material name="Grey">
+                <color rgba="0.7 0.7 0.7 1"/>
+            </material>
+        </visual>
     </link>
 <!--=================== JOINTS ========================-->
@@ -207,7 +234,13 @@
         <axis xyz = "0 0 1"/>
         <limit lower = "-3.1067" upper = "3.1067" effort = "50" velocity = "10"/>
-        <origin rpy="1.57075 0 0" xyz = "0 0 0"/>
+        <origin rpy="1.57075 0 0" xyz = "0 -0.043 0"/>
+        <!-- <origin rpy="1.57075 0 0" xyz = "0 0 0"/> -->
         <dynamics damping="0"/>
     </joint>
+    <joint name="joint_6_to_tool" type="fixed">
+        <parent link="link_6"/>
+        <child link="tool"/>
+        <origin rpy="0 0 0" xyz = "0 0 0.0805"/>
+    </joint>
     <transmission name="tran1">
         <type>transmission_interface/SimpleTransmission</type>

Commit message: finalize path planner

File: emu_description/urdf/emu.xacro (robot description, xacro)
@@ -194,5 +194,5 @@
         <child link="link_1"/>
         <axis xyz = "0 0 1"/>
-        <limit lower = "-3.1066" upper = "3.1066" effort = "1000" velocity = "1000"/>
+        <limit lower = "-3.1066" upper = "3.1066" effort = "1000" velocity = "2.5" acceleration = "1"/>
         <dynamics damping="0.1"/>
     </joint>
@@ -201,5 +201,5 @@
         <child link="link_2"/>
         <axis xyz = "0 0 1"/>
-        <limit lower = "-2.917" upper = "1.703" effort = "1000" velocity = "1000"/>
+        <limit lower = "-2.917" upper = "1.703" effort = "1000" velocity = "1.5" acceleration = "1"/>
         <origin rpy="1.57075 0 0" xyz = "0.12596 0 0.30767"/>
         <dynamics damping="0.1"/>
@@ -209,5 +209,5 @@
         <child link="link_3"/>
         <axis xyz = "0 0 1"/>
-        <limit lower = "-1.4312" upper = "4.1190" effort = "1000" velocity = "1000"/>
+        <limit lower = "-1.4312" upper = "4.1190" effort = "1000" velocity = "2.5" acceleration = "1"/>
         <origin rpy="0 0 1.57075" xyz = "0 0.4 0"/>
         <dynamics damping="0.1"/>
@@ -217,5 +217,5 @@
         <child link="link_4"/>
         <axis xyz = "0 0 1"/>
-        <limit lower = "-3.1067" upper = "3.1067" effort = "1000" velocity = "1000"/>
+        <limit lower = "-3.1067" upper = "3.1067" effort = "1000" velocity = "1.5" acceleration = "2"/>
         <origin rpy="1.57075 0 0" xyz = "0.05 0 0"/>
         <dynamics damping="0.03"/>
@@ -225,5 +225,5 @@
         <child link="link_5"/>
         <axis xyz = "0 0 1"/>
-        <limit lower = "-3.1067" upper = "3.1067" effort = "1000" velocity = "1000"/>
+        <limit lower = "-3.1067" upper = "3.1067" effort = "1000" velocity = "2" acceleration = "2"/>
         <origin rpy="-1.57075 0 0" xyz = "0 0 0.466"/>
         <dynamics damping="0.01"/>
@@ -233,5 +233,5 @@
         <child link="link_6"/>
         <axis xyz = "0 0 1"/>
-        <limit lower = "-3.1067" upper = "3.1067" effort = "50" velocity = "10"/>
+        <limit lower = "-3.1067" upper = "3.1067" effort = "50" velocity = "2" acceleration = "2"/>
         <origin rpy="1.57075 0 0" xyz = "0 -0.043 0"/>
         <!-- <origin rpy="1.57075 0 0" xyz = "0 0 0"/> -->
