Commit message: add gripper to the planner

File: emu_description/urdf/emu.xacro (robot description, xacro)
@@ -163,5 +163,5 @@
         </visual>
     </link>
-    <link name="tool">
+    <link name="tool_base">
 		<inertial>
 			<origin xyz = "-0.00016738 0 0.04413320"/>
@@ -172,16 +172,34 @@
 			<origin xyz="0 0 0"/>
 			<geometry>
-				<mesh filename="package://emu_description/meshes/tool_joulin.STL" scale="1 1 1"/>
-			</geometry>
-		</collision>
-        <visual>
-            <geometry>
-                <mesh filename="package://emu_description/meshes/tool_joulin.STL" scale="1 1 1"/>
-            </geometry>
-            <material name="Grey">
-                <color rgba="0.7 0.7 0.7 1"/>
-            </material>
-        </visual>
-    </link>
+				<mesh filename="package://emu_description/meshes/tool_static.STL" scale="1 1 1"/>
+			</geometry>
+		</collision>
+        <visual>
+            <geometry>
+                <mesh filename="package://emu_description/meshes/tool_static.STL" scale="1 1 1"/>
+            </geometry>
+            <material name="Grey">
+                <color rgba="0.7 0.7 0.7 1"/>
+            </material>
+        </visual>
+    </link>
+    <link name="sliding_jaw">
+        <collision>
+			<origin xyz="0 0 0"/>
+			<geometry>
+				<mesh filename="package://emu_description/meshes/tool_sliding.STL" scale="1 1 1"/>
+			</geometry>
+		</collision>
+        <visual>
+            <geometry>
+                <mesh filename="package://emu_description/meshes/tool_sliding.STL" scale="1 1 1"/>
+            </geometry>
+            <material name="Grey">
+                <color rgba="0.7 0.7 0.7 1"/>
+            </material>
+        </visual>
+    </link>
+    <link name="grasp_frame"/>
+    <link name="suction_frame"/>
 <!--=================== JOINTS ========================-->
     <!-- <joint name="world_to_base" type="fixed">
@@ -238,8 +256,27 @@
         <dynamics damping="0"/>
     </joint>
-    <joint name="joint_6_to_tool" type="fixed">
+    <joint name="joint_6_to_tool_base" type="fixed">
         <parent link="link_6"/>
-        <child link="tool"/>
-        <origin rpy="0 0 0" xyz = "0 0 0.0805"/>
+        <child link="tool_base"/>
+        <origin rpy="0 0 0" xyz = "0 0 0"/>
+    </joint>
+    <joint name="sliding_jaw_joint" type="prismatic">
+        <parent link="tool_base"/>
+        <child link="sliding_jaw"/>
+        <axis xyz = "0 0 1"/>
+        <limit lower = "0" upper = "0.0715" effort = "10" velocity = "5" acceleration = "10"/>
+        <origin rpy="1.57075 0 0" xyz = "0 0.0288 0.145"/>
+    </joint>
+    <joint name="grasp_frame_transform" type="fixed">
+        <parent link="tool_base"/>
+        <child link="grasp_frame"/>
+        <axis xyz = "0 0 1"/>
+        <origin rpy="0 0 0" xyz = "0 0 0.145"/>
+    </joint>
+    <joint name="suction_frame_transform" type="fixed">
+        <parent link="tool_base"/>
+        <child link="suction_frame"/>
+        <axis xyz = "0 0 1"/>
+        <origin rpy="0 0 0" xyz = "0 -0.0881 0.1852"/>
     </joint>
     <transmission name="tran1">

Commit message: Improve planner

File: emu_description/urdf/emu.xacro (robot description, xacro)
@@ -12,9 +12,9 @@
     <!-- <link name="world"/> -->
     <link name="base_link">
-		<inertial>
+		<!-- <inertial>
 			<origin xyz = "0.03581298 0.00000140 0.07057116"/>
 			<mass value = "4.6883"/>
 			<inertia ixx = "0.02107003" iyy = "0.04864817" izz = "0.05239187" ixy = "0.00000013" ixz = "0.0149951" iyz = "-0.00000032"/>
-		</inertial>
+		</inertial> -->
         <collision>
 			<origin xyz="0 0 0"/>

Commit message: add new gripper finger

File: emu_description/urdf/emu.xacro (robot description, xacro)
@@ -172,10 +172,10 @@
 			<origin xyz="0 0 0"/>
 			<geometry>
-				<mesh filename="package://emu_description/meshes/tool_static.STL" scale="1 1 1"/>
-			</geometry>
-		</collision>
-        <visual>
-            <geometry>
-                <mesh filename="package://emu_description/meshes/tool_static.STL" scale="1 1 1"/>
+				<mesh filename="package://emu_description/meshes/tool_static.dae" scale="1 1 1"/>
+			</geometry>
+		</collision>
+        <visual>
+            <geometry>
+                <mesh filename="package://emu_description/meshes/tool_static.dae" scale="1 1 1"/>
             </geometry>
             <material name="Grey">
@@ -188,10 +188,10 @@
 			<origin xyz="0 0 0"/>
 			<geometry>
-				<mesh filename="package://emu_description/meshes/tool_sliding.STL" scale="1 1 1"/>
-			</geometry>
-		</collision>
-        <visual>
-            <geometry>
-                <mesh filename="package://emu_description/meshes/tool_sliding.STL" scale="1 1 1"/>
+				<mesh filename="package://emu_description/meshes/tool_sliding.dae" scale="1 1 1"/>
+			</geometry>
+		</collision>
+        <visual>
+            <geometry>
+                <mesh filename="package://emu_description/meshes/tool_sliding.dae" scale="1 1 1"/>
             </geometry>
             <material name="Grey">
@@ -266,5 +266,5 @@
         <axis xyz = "0 0 1"/>
         <limit lower = "0" upper = "0.0715" effort = "10" velocity = "5" acceleration = "10"/>
-        <origin rpy="1.57075 0 0" xyz = "0 0.0288 0.145"/>
+        <origin rpy="1.57075 0 0" xyz = "0 0.0178 0.1205"/>
     </joint>
     <joint name="grasp_frame_transform" type="fixed">
@@ -272,5 +272,5 @@
         <child link="grasp_frame"/>
         <axis xyz = "0 0 1"/>
-        <origin rpy="0 0 0" xyz = "0 0 0.145"/>
+        <origin rpy="0 0 0" xyz = "0 -0.033 0.1205"/>
     </joint>
     <joint name="suction_frame_transform" type="fixed">
@@ -278,5 +278,5 @@
         <child link="suction_frame"/>
         <axis xyz = "0 0 1"/>
-        <origin rpy="0 0 0" xyz = "0 -0.0881 0.1852"/>
+        <origin rpy="0 0 0" xyz = "0 -0.0923 0.1602"/>
     </joint>
     <transmission name="tran1">

Commit message: night before demo2

File: emu_description/urdf/emu.xacro (robot description, xacro)
@@ -227,5 +227,5 @@
         <child link="link_3"/>
         <axis xyz = "0 0 1"/>
-        <limit lower = "-1.4312" upper = "4.1190" effort = "1000" velocity = "2.5" acceleration = "1"/>
+        <limit lower = "-1.4312" upper = "1.6" effort = "1000" velocity = "2.5" acceleration = "1"/>
         <origin rpy="0 0 1.57075" xyz = "0 0.4 0"/>
         <dynamics damping="0.1"/>
@@ -266,5 +266,5 @@
         <axis xyz = "0 0 1"/>
         <limit lower = "0" upper = "0.0715" effort = "10" velocity = "5" acceleration = "10"/>
-        <origin rpy="1.57075 0 0" xyz = "0 0.0178 0.1205"/>
+        <origin rpy="1.57075 0 0" xyz = "0 0.0178 0.1095"/>
     </joint>
     <joint name="grasp_frame_transform" type="fixed">
@@ -272,5 +272,5 @@
         <child link="grasp_frame"/>
         <axis xyz = "0 0 1"/>
-        <origin rpy="0 0 0" xyz = "0 -0.033 0.1205"/>
+        <origin rpy="0 0 0" xyz = "0 -0.033 0.1095"/>
     </joint>
     <joint name="suction_frame_transform" type="fixed">
@@ -278,5 +278,5 @@
         <child link="suction_frame"/>
         <axis xyz = "0 0 1"/>
-        <origin rpy="0 0 0" xyz = "0 -0.0923 0.1602"/>
+        <origin rpy="0 0 0" xyz = "0 -0.0923 0.1492"/>
     </joint>
     <transmission name="tran1">
